File: coil_test_circuit/coil_test_circuit.kicad_sch (KiCad schematic)
At the start: 9 parts, among them J1 COIL, SW1 SW_Push_SPDT

Commit message: Schematic cleanup
Connections:
- net at A1.27 (+5V), R1.1, R2.1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: no longer R3.1, SW1.1 (A)
- new net: R3.1, SW1.1 (A)
Changed lines of the file:
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@@
   (junction (at 124.46 134.62) (diameter 0) (color 0 0 0 0)
-  )
-  (junction (at 124.46 99.06) (diameter 0) (color 0 0 0 0)
-  )
-  (junction (at 124.46 104.14) (diameter 0) (color 0 0 0 0)
   )
   (junction (at 209.55 134.62) (diameter 0) (color 0 0 0 0)
@@
   )
   (wire (pts (xy 142.24 121.92) (xy 148.59 121.92))
-    (stroke (width 0) (type default))
-  )
-  (wire (pts (xy 63.5 91.44) (xy 71.12 91.44))
-    (stroke (width 0) (type default))
-  )
-  (wire (pts (xy 124.46 104.14) (xy 124.46 99.06))
     (stroke (width 0) (type default))
   )
@@
   )
   (wire (pts (xy 209.55 97.79) (xy 209.55 67.31))
+    (stroke (width 0) (type default))
+  )
+  (wire (pts (xy 68.58 91.44) (xy 71.12 91.44))
     (stroke (width 0) (type default))
   )
@@
     )
   )
-  (global_label "TRIGGER" (shape input) (at 63.5 91.44 180) (fields_autoplaced)
+  (global_label "TRIGGER" (shape input) (at 68.58 91.44 180) (fields_autoplaced)
     (effects (font (size 1.27 1.27)) (justify right))
-    (property "Intersheetrefs" "${INTERSHEET_REFS}" (at 52.7134 91.44 0)
+    (property "Intersheetrefs" "${INTERSHEET_REFS}" (at 57.7934 91.44 0)
       (effects (font (size 1.27 1.27)) (justify right) hide)
     )
